File: wifi-nunchuck/wifi-nunchuck.kicad_pcb (KiCad board)
At the start: 2 copper layers, 14.6 x 8 mm, 22 parts, among them J2 USB_B_Micro, Q1 BSS138, Q2 BSS138, U1 ESP32-WROOM-32, U2 AMS1117-3.3, U3 CH340C

Commit message: pcb wiring
Parts:
- moved R3 56.5 mm to (85.3, 72.9), turned to -90 degrees
- moved R4 53.7 mm to (87.0, 72.9), turned to 90 degrees
- moved R2 52.1 mm to (93.6, 72.9), turned to 90 degrees
- moved C3 48.1 mm to (90.3, 72.9), turned to 90 degrees
- moved R5 47.7 mm to (103.9, 82.9), turned to 90 degrees
- moved C4 47.7 mm to (88.6, 72.9), turned to 90 degrees
- moved C1 47.5 mm to (96.8, 72.9), turned to 90 degrees
- moved R6 44.8 mm to (105.5, 82.9), turned to 90 degrees
- moved C5 43.5 mm to (91.9, 72.9), turned to 90 degrees
- moved D2 42.9 mm to (82.5, 63.9)
- moved D1 42.9 mm to (82.5, 62.0)
- moved R1 39.5 mm to (95.1, 72.9), turned to -90 degrees
- moved C2 39.2 mm to (87.8, 48.3), turned to 90 degrees
- moved Q2 20.9 mm to (86.2, 76.7), turned to 90 degrees
- moved EN1 18.0 mm to (103.9, 74.3), turned to 180 degrees
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Routing:
- net +3V3: track 0.00 -> 93.7 mm, vias 0 -> 1
- net RX-PROG: track 0.00 -> 46.9 mm, vias 0 -> 2
- net TX-PROG: track 0.00 -> 46.8 mm, vias 0 -> 2
- net SCL: track 0.00 -> 44.1 mm, vias 0 -> 2
- net ESP32_EN: track 0.00 -> 44.0 mm, vias 0 -> 4
- net SDA: track 0.00 -> 41.2 mm, vias 0 -> 2
- net ESP32_IO0: track 0.00 -> 28.1 mm
- net Net-(U1-IO13): track 0.00 -> 16.6 mm, vias 0 -> 2
- net Net-(U1-IO12): track 0.00 -> 16.0 mm
- net Net-(D1-A): track 0.00 -> 14.3 mm, vias 0 -> 2
- net Net-(D2-A): track 0.00 -> 13.9 mm, vias 0 -> 2
- net Net-(Q1-S): track 0.00 -> 13.3 mm
- net D+: track 0.00 -> 8.33 mm
- net D-: track 0.00 -> 8.13 mm
- net Net-(Q1-G): track 0.00 -> 5.54 mm
Other:
- board size 14.6 x 8 mm -> 29.7 x 47.8 mm

Commit message: add gnd plane
Routing:
- added copper zone on B.Cu, net GND
- added copper zone on F.Cu, net GND
Changed lines of the file:
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@@
 		(tags "SPST button tactile switch")
 		(property "Reference" "EN1"
-			(at 0 -2.6 360)
+			(at 0 -2.6 0)
 			(layer "F.SilkS")
 			(effects
@@
 		)
 		(property "Value" "SW_Push"
-			(at 0 3 360)
+			(at 0 3 0)
 			(layer "F.Fab")
 			(effects
@@
 		)
 		(fp_text user "${REFERENCE}"
-			(at 0 -2.6 360)
+			(at 0 -2.6 0)
 			(layer "F.Fab")
 			(effects
@@
 		(tags "LED")
 		(property "Reference" "D2"
-			(at 2.413 0 360)
+			(at 2.413 0 0)
 			(layer "F.SilkS")
 			(effects
@@
 		)
 		(property "Value" "LED"
-			(at 0 1.43 360)
+			(at 0 1.43 0)
 			(layer "F.Fab")
 			(effects
@@
 		)
 		(fp_text user "${REFERENCE}"
-			(at 0 0 360)
+			(at 0 0 0)
 			(layer "F.Fab")
 			(effects
@@
 		(tags "Nintendo Wii Nunchuck I2C PCB")
 		(property "Reference" "U4"
-			(at -6.858 3.048 360)
+			(at -6.858 3.048 0)
 			(layer "F.SilkS")
 			(effects
@@
 		)
 		(property "Value" "~"
-			(at 1.9 5 360)
+			(at 1.9 5 0)
 			(layer "F.Fab")
 			(effects
@@
 		)
 		(fp_text user "${REFERENCE}"
-			(at 1.9 -1.2 360)
+			(at 1.9 -1.2 0)
 			(layer "F.Fab")
 			(effects
@@
 		(net 44)
 	)
+	(zone
+		(net 1)
+		(net_name "GND")
+		(layers "F&B.Cu")
+		(hatch edge 0.5)
+		(connect_pads
+			(clearance 0.5)
+		)
+		(min_thickness 0.25)
+		(filled_areas_thickness no)
+		(fill yes
+			(thermal_gap 0.5)
+			(thermal_bridge_width 0.5)
+		)
+		(polygon
+			(pts
+				(xy 80 44) (xy 111 44) (xy 111 95) (xy 80 95)
+			)
+		)
+	)
 )

Commit message: update gnd
Routing:
- net +5V: track 0.00 -> 29.7 mm, vias 0 -> 2
- net GND: track 0.00 -> 4.75 mm, vias 0 -> 21
